File: Eagle/blt_20221101.brd (EAGLE design)
At the start: 29.8 x 35.6 mm, 20 parts, among them IC1 74HC4066D, IC2 74HC4066D, IC3 ATTINY84V-10SSUR

Commit message: Add files via upload
Connections:
- net GND: now also IC3.14
Changed lines of the file:
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@@
 <drawing>
 <settings>
-<setting alwaysvectorfont="no"/>
+<setting alwaysvectorfont="yes"/>
 <setting verticaltext="up"/>
 </settings>
@@
 <via x="10.31875" y="24.765" extent="1-16" drill="0.35"/>
 <via x="6.50875" y="21.59" extent="1-16" drill="0.35"/>
+<contactref element="IC3" pad="14"/>
 </signal>
 <signal name="EN_NG">
@@
 </signals>
 <mfgpreviewcolors>
-<mfgpreviewcolor name="soldermaskcolor" color="0xC8008000"/>
+<mfgpreviewcolor name="soldermaskcolor" color="0xC80055FF"/>
 <mfgpreviewcolor name="silkscreencolor" color="0xFFFEFEFE"/>
 <mfgpreviewcolor name="backgroundcolor" color="0xFF282828"/>
-<mfgpreviewcolor name="coppercolor" color="0xFFFFBF00"/>
+<mfgpreviewcolor name="coppercolor" color="0xFFD8D8D8"/>
 <mfgpreviewcolor name="substratecolor" color="0xFF786E46"/>
 </mfgpreviewcolors>
